File: Smart Card Test Board/dpMaster.brd (EAGLE design)
At the start: 68.2 x 45.7 mm, 6 parts, among them J1 22-27-2021-02

Commit message: Board v3
Parts:
- added C1: (no value), capacitor-wima:C5B4.5
- moved U$2 1.27 mm to (16.5, 5.08)
Connections:
- net N$14: now also C1.1
- net N$6: now also C1.2
Routing:
- net N$6: track 50.8 -> 53.3 mm
- net N$14: track 171.7 -> 173.0 mm
Other:
- board size 68.2 x 45.7 mm -> 68.2 x 43.2 mm
Changed lines of the file:
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@@
 <layer number="43" name="vRestrict" color="2" fill="10" visible="yes" active="yes"/>
 <layer number="44" name="Drills" color="7" fill="1" visible="no" active="yes"/>
-<layer number="45" name="Holes" color="7" fill="1" visible="no" active="yes"/>
+<layer number="45" name="Holes" color="7" fill="1" visible="yes" active="yes"/>
 <layer number="46" name="Milling" color="3" fill="1" visible="no" active="yes"/>
 <layer number="47" name="Measures" color="7" fill="1" visible="no" active="yes"/>
@@
 <board>
 <plain>
-<wire x1="2.54" y1="0" x2="70.79" y2="0" width="0" layer="20"/>
-<wire x1="70.79" y1="0" x2="70.79" y2="45.71" width="0" layer="20"/>
-<wire x1="70.79" y1="45.71" x2="2.54" y2="45.71" width="0" layer="20"/>
-<wire x1="2.54" y1="45.71" x2="2.54" y2="0" width="0" layer="20"/>
+<wire x1="2.54" y1="0" x2="70.79" y2="0" width="0.254" layer="20"/>
+<wire x1="70.79" y1="0" x2="70.79" y2="43.17" width="0.254" layer="20"/>
+<wire x1="70.79" y1="43.17" x2="2.54" y2="43.17" width="0.6096" layer="20"/>
+<wire x1="2.54" y1="43.17" x2="2.54" y2="0" width="0.254" layer="20"/>
 </plain>
 <attributes>
@@
 </element>
 <element name="U$1" library="sfc-120-t2-l-d" package="SFC-120-T2-L-D" value="SFC-120-T2-L-D" x="16.51" y="33.02"/>
-<element name="U$2" library="sfc-120-t2-l-d" package="SFC-120-T2-L-D" value="SFC-120-T2-L-D" x="16.51" y="6.35"/>
+<element name="U$2" library="sfc-120-t2-l-d" package="SFC-120-T2-L-D" value="SFC-120-T2-L-D" x="16.51" y="5.08"/>
+<element name="C1" library="capacitor-wima" package="C5B4.5" value="" x="57.15" y="5.08" rot="R270"/>
 </elements>
 <signals>
@@
 <contactref element="U$1" pad="P$12"/>
 <wire x1="22.86" y1="35.56" x2="22.86" y2="33.02" width="0" layer="19" extent="1-16"/>
-<wire x1="62.23" y1="19.05" x2="66.04" y2="19.05" width="0.8128" layer="16"/>
-<wire x1="66.04" y1="19.05" x2="66.04" y2="40.64" width="0.8128" layer="16"/>
-<wire x1="66.04" y1="40.64" x2="22.86" y2="40.64" width="0.8128" layer="16"/>
-<wire x1="22.86" y1="40.64" x2="22.86" y2="39.37" width="0.8128" layer="16"/>
+<wire x1="62.23" y1="19.05" x2="66.04" y2="19.05" width="1.016" layer="16"/>
+<wire x1="66.04" y1="19.05" x2="66.04" y2="40.64" width="1.016" layer="16"/>
+<wire x1="66.04" y1="40.64" x2="22.86" y2="40.64" width="1.016" layer="16"/>
+<wire x1="22.86" y1="40.64" x2="22.86" y2="39.37" width="1.016" layer="16"/>
 <wire x1="22.86" y1="39.37" x2="22.86" y2="33.02" width="0" layer="19" extent="1-16"/>
 </signal>
@@
 <contactref element="U$2" pad="P$1"/>
 <contactref element="J1" pad="2"/>
-<wire x1="62.23" y1="6.35" x2="62.23" y2="2.54" width="0.8128" layer="16"/>
-<wire x1="62.23" y1="2.54" x2="16.51" y2="2.54" width="0.8128" layer="16"/>
-<wire x1="16.51" y1="6.35" x2="16.51" y2="5.08" width="0" layer="19" extent="1-16"/>
-<wire x1="16.51" y1="2.54" x2="16.51" y2="3.81" width="0.8128" layer="16"/>
-<wire x1="16.51" y1="3.81" x2="16.51" y2="5.08" width="0" layer="19" extent="1-16"/>
+<wire x1="62.23" y1="6.35" x2="62.23" y2="1.27" width="1.016" layer="16"/>
+<wire x1="62.23" y1="1.27" x2="57.15" y2="1.27" width="1.016" layer="16"/>
+<wire x1="57.15" y1="1.27" x2="16.51" y2="1.27" width="1.016" layer="16"/>
+<wire x1="16.51" y1="1.27" x2="16.51" y2="2.54" width="1.016" layer="16"/>
+<contactref element="C1" pad="2"/>
+<wire x1="57.15" y1="2.54" x2="57.15" y2="1.27" width="1.016" layer="16"/>
+<wire x1="16.51" y1="3.81" x2="16.51" y2="5.08" width="0" layer="19" extent="1-1"/>
+<wire x1="16.51" y1="2.54" x2="16.51" y2="3.81" width="0" layer="19" extent="16-16"/>
 </signal>
 <signal name="N$8">
@@
 <contactref element="SV1" pad="4"/>
 <contactref element="D1" pad="A"/>
-<wire x1="62.23" y1="24.13" x2="57.15" y2="24.13" width="0.8128" layer="16"/>
-<wire x1="21.59" y1="20.32" x2="54.61" y2="20.32" width="0.8128" layer="16"/>
-<wire x1="54.61" y1="20.32" x2="57.15" y2="20.32" width="0.8128" layer="16"/>
-<wire x1="57.15" y1="20.32" x2="57.15" y2="24.13" width="0.8128" layer="16"/>
-<wire x1="21.59" y1="20.32" x2="21.59" y2="30.48" width="0.8128" layer="16"/>
+<wire x1="62.23" y1="24.13" x2="57.15" y2="24.13" width="1.016" layer="16"/>
+<wire x1="21.59" y1="20.32" x2="54.61" y2="20.32" width="1.016" layer="16"/>
+<wire x1="54.61" y1="20.32" x2="57.15" y2="20.32" width="1.016" layer="16"/>
+<wire x1="57.15" y1="20.32" x2="57.15" y2="24.13" width="1.016" layer="16"/>
+<wire x1="21.59" y1="20.32" x2="21.59" y2="30.48" width="1.016" layer="16"/>
 <wire x1="21.59" y1="30.48" x2="21.59" y2="31.75" width="0" layer="19" extent="1-16"/>
 </signal>
@@
 <contactref element="U$1" pad="P$10"/>
 <contactref element="D1" pad="C"/>
-<wire x1="57.15" y1="13.97" x2="13.97" y2="13.97" width="0.8128" layer="16"/>
-<wire x1="13.97" y1="13.97" x2="13.97" y2="34.925" width="0.8128" layer="16"/>
-<wire x1="13.97" y1="34.925" x2="21.59" y2="34.925" width="0.8128" layer="16"/>
-<wire x1="21.59" y1="34.925" x2="21.59" y2="34.29" width="0.8128" layer="16"/>
+<wire x1="57.15" y1="13.97" x2="13.97" y2="13.97" width="1.016" layer="16"/>
+<wire x1="13.97" y1="13.97" x2="13.97" y2="34.925" width="1.016" layer="16"/>
+<wire x1="13.97" y1="34.925" x2="21.59" y2="34.925" width="1.016" layer="16"/>
+<wire x1="21.59" y1="34.925" x2="21.59" y2="34.29" width="1.016" layer="16"/>
 <wire x1="21.59" y1="34.29" x2="21.59" y2="33.02" width="0" layer="19" extent="1-16"/>
 </signal>
@@
 <contactref element="U$1" pad="P$11"/>
 <contactref element="SV1" pad="7"/>
-<wire x1="62.23" y1="16.51" x2="22.86" y2="16.51" width="0.8128" layer="16"/>
-<wire x1="22.86" y1="16.51" x2="22.86" y2="17.78" width="0.8128" layer="16"/>
+<wire x1="62.23" y1="16.51" x2="22.86" y2="16.51" width="1.016" layer="16"/>
+<wire x1="22.86" y1="16.51" x2="22.86" y2="17.78" width="1.016" layer="16"/>
 <wire x1="22.86" y1="17.78" x2="22.86" y2="31.75" width="0" layer="19" extent="1-16"/>
 </signal>
@@
 <contactref element="SV1" pad="2"/>
 <contactref element="R1" pad="2"/>
-<wire x1="62.23" y1="29.21" x2="53.34" y2="29.21" width="0.8128" layer="16"/>
-<wire x1="53.34" y1="29.21" x2="53.34" y2="24.13" width="0.4064" layer="16"/>
-<wire x1="53.34" y1="24.13" x2="24.13" y2="24.13" width="0.8128" layer="16"/>
-<wire x1="54.61" y1="33.02" x2="53.34" y2="33.02" width="0.8128" layer="16"/>
-<wire x1="53.34" y1="33.02" x2="53.34" y2="24.13" width="0.8128" layer="16"/>
-<wire x1="24.13" y1="24.13" x2="24.13" y2="30.48" width="0.8128" layer="16"/>
+<wire x1="62.23" y1="29.21" x2="53.34" y2="29.21" width="1.016" layer="16"/>
+<wire x1="53.34" y1="29.21" x2="53.34" y2="24.13" width="1.016" layer="16"/>
+<wire x1="53.34" y1="24.13" x2="24.13" y2="24.13" width="1.016" layer="16"/>
+<wire x1="54.61" y1="33.02" x2="53.34" y2="33.02" width="1.016" layer="16"/>
+<wire x1="53.34" y1="33.02" x2="53.34" y2="24.13" width="1.016" layer="16"/>
+<wire x1="24.13" y1="24.13" x2="24.13" y2="30.48" width="1.016" layer="16"/>
 <wire x1="24.13" y1="30.48" x2="24.13" y2="31.75" width="0" layer="19" extent="1-16"/>
 </signal>
@@
 <contactref element="SV1" pad="1"/>
 <contactref element="J1" pad="1"/>
-<wire x1="26.67" y1="27.94" x2="50.8" y2="27.94" width="0.8128" layer="16"/>
-<wire x1="50.8" y1="27.94" x2="50.8" y2="36.83" width="0.8128" layer="16"/>
-<wire x1="50.8" y1="36.83" x2="62.23" y2="36.83" width="0.8128" layer="16"/>
-<wire x1="62.23" y1="36.83" x2="62.23" y2="31.75" width="0.8128" layer="16"/>
-<wire x1="26.67" y1="27.94" x2="25.4" y2="30.48" width="0.8128" layer="16"/>
-<wire x1="40.64" y1="8.89" x2="11.43" y2="8.89" width="0.8128" layer="16"/>
-<wire x1="11.43" y1="8.89" x2="11.43" y2="36.83" width="0.8128" layer="16"/>
-<wire x1="11.43" y1="36.83" x2="50.8" y2="36.83" width="0.8128" layer="16"/>
+<wire x1="26.67" y1="27.94" x2="50.8" y2="27.94" width="1.016" layer="16"/>
+<wire x1="50.8" y1="27.94" x2="50.8" y2="36.83" width="1.016" layer="16"/>
+<wire x1="50.8" y1="36.83" x2="62.23" y2="36.83" width="1.016" layer="16"/>
+<wire x1="62.23" y1="36.83" x2="62.23" y2="31.75" width="1.016" layer="16"/>
+<wire x1="26.67" y1="27.94" x2="25.4" y2="30.48" width="1.016" layer="16"/>
+<wire x1="40.64" y1="8.89" x2="11.43" y2="8.89" width="1.016" layer="16"/>
+<wire x1="11.43" y1="8.89" x2="11.43" y2="36.83" width="1.016" layer="16"/>
+<wire x1="11.43" y1="36.83" x2="50.8" y2="36.83" width="1.016" layer="16"/>
+<wire x1="62.23" y1="8.89" x2="57.15" y2="8.89" width="1.016" layer="16"/>
+<wire x1="57.15" y1="8.89" x2="40.64" y2="8.89" width="1.016" layer="16"/>
+<wire x1="40.64" y1="8.89" x2="40.64" y2="7.62" width="1.016" layer="16"/>
+<contactref element="C1" pad="1"/>
+<wire x1="57.15" y1="7.62" x2="57.15" y2="8.89" width="1.016" layer="16"/>
 <wire x1="25.4" y1="30.48" x2="25.4" y2="31.75" width="0" layer="19" extent="16-16"/>
-<wire x1="40.64" y1="5.08" x2="40.64" y2="6.35" width="0" layer="19" extent="1-1"/>
-<wire x1="40.64" y1="7.62" x2="40.64" y2="6.35" width="0" layer="19" extent="1-16"/>
-<wire x1="62.23" y1="8.89" x2="40.64" y2="8.89" width="0.8128" layer="16"/>
-<wire x1="40.64" y1="8.89" x2="40.64" y2="7.62" width="0.8128" layer="16"/>
-<wire x1="40.64" y1="7.62" x2="40.64" y2="6.35" width="0" layer="19" extent="1-16"/>
+<wire x1="40.64" y1="5.08" x2="40.64" y2="7.62" width="0" layer="19" extent="16-16"/>
+<wire x1="40.64" y1="3.81" x2="40.64" y2="5.08" width="0" layer="19" extent="1-1"/>
 </signal>
 </signals>
